Commit message: Tweaked wheel physics slightly to make Audibot less prone to sliding

File: audibot_description/urdf/audibot.urdf.xacro (robot description, xacro)
@@ -6,5 +6,5 @@
   <xacro:property name="wheel_radius" value="0.36" />
   <xacro:property name="wheel_thickness" value="0.25" />
-  <xacro:property name="wheel_mass" value="20.0" />
+  <xacro:property name="wheel_mass" value="40.0" />
   <xacro:property name="body_mass" value="1620.0" />
   <xacro:property name="body_width" value="${2*half_rear_track_width}" />
@@ -154,5 +154,5 @@
   <xacro:front_wheel name="fl" x="${half_wheelbase}" y="${half_front_track_width}" z="0" flip="1" />
   <xacro:front_wheel name="fr" x="${half_wheelbase}" y="${-half_front_track_width}" z="0" flip="0" />
-  <xacro:property name="wheel_friction" value="1.5" />
+  <xacro:property name="wheel_friction" value="1.75" />
   <gazebo reference="base_link" >
     <mu1>0.5</mu1>

Commit message: Removes logo from the hood
Transparent backgrounds in textures don't look right in Rviz

File: audibot_description/urdf/audibot.urdf.xacro (robot description, xacro)
@@ -127,12 +127,4 @@
     </inertial>
   </link>
-  <link name="hood_logo" >
-    <visual>
-      <origin xyz="0.035 0 0.025" rpy="0 0 0" />
-      <geometry>
-        <mesh filename="package://audibot_description/meshes/hood_logo.dae" scale="1.01 1.01 1.01" />
-      </geometry>
-    </visual>
-  </link>
   <joint name="base_link" type="fixed">
     <origin xyz="${half_wheelbase} 0 ${wheel_radius}" rpy="0 0 0"/>
@@ -140,14 +132,4 @@
     <child link="base_link"/>
   </joint>
-  <joint name="hood_logo" type="fixed" >
-    <parent link="base_link" />
-    <child link="hood_logo" />
-    <origin xyz="0 0 0" rpy="0 0 0" />
-  </joint>
-  <gazebo reference="hood_logo" >
-    <visual>
-      <transparency>0.01</transparency>
-    </visual>
-  </gazebo>
   <xacro:rear_wheel name="rl" x="${-half_wheelbase}" y="${half_rear_track_width}" z="0" flip="1" />
   <xacro:rear_wheel name="rr" x="${-half_wheelbase}" y="${-half_rear_track_width}" z="0" flip="0" />

Commit message: Changes names of joints to be different from links
Gazebo 11 doesn't let joint names and link names be the same, which was allowed in earlier versions

File: audibot_description/urdf/audibot.urdf.xacro (robot description, xacro)
@@ -27,5 +27,5 @@
         </xacro:if>
         <jointName>
-            steer_fl, steer_fr, wheel_fl, wheel_fr, wheel_rl, wheel_rr
+            steer_fl_joint, steer_fr_joint, wheel_fl_joint, wheel_fr_joint, wheel_rl_joint, wheel_rr_joint
         </jointName>
         <updateRate>100</updateRate>
@@ -52,5 +52,5 @@
       </inertial>
     </link>
-    <joint name="wheel_${name}" type="continuous" >
+    <joint name="wheel_${name}_joint" type="continuous" >
       <parent link="base_link" />
       <child link="wheel_${name}" />
@@ -86,5 +86,5 @@
       </inertial>
     </link>
-    <joint name="steer_${name}" type="revolute" >
+    <joint name="steer_${name}_joint" type="revolute" >
       <parent link="base_link" />
       <child link="steer_${name}" />
@@ -93,5 +93,5 @@
       <limit upper="0.6" lower="-0.6" effort="0.0" velocity="0.0" />
     </joint>
-    <joint name="wheel_${name}" type="continuous" >
+    <joint name="wheel_${name}_joint" type="continuous" >
       <parent link="steer_${name}" />
       <child link="wheel_${name}" />
@@ -127,5 +127,5 @@
     </inertial>
   </link>
-  <joint name="base_link" type="fixed">
+  <joint name="base_link_joint" type="fixed">
     <origin xyz="${half_wheelbase} 0 ${wheel_radius}" rpy="0 0 0"/>
     <parent link="base_footprint"/>

Commit message: Implements tf_prefix functionality that was removed from robot_state_publisher
Necessary to support multiple instances of Audibot without colliding TF frame IDs. There are PRs open to re-enable the tf_prefix functionality, but none merged in yet:

https://github.com/ros/robot_state_publisher/pull/127/

https://github.com/ros/robot_state_publisher/pull/139

File: audibot_description/urdf/audibot.urdf.xacro (robot description, xacro)
@@ -13,5 +13,4 @@
   <xacro:arg name="pub_tf" default="true" />
   <xacro:arg name="robot_name" default="" />
-  <xacro:property name="robot_name_prop" value="$(arg robot_name)" />
   <gazebo>
     <!-- Simulated vehicle interface -->
@@ -23,12 +22,8 @@
     <!-- Publish current joint angles -->
     <plugin name="joint_state_publisher" filename="libgazebo_ros_joint_state_publisher.so">
-        <xacro:if value="${robot_name_prop != ''}" >
-          <robotNamespace>$(arg robot_name)</robotNamespace>
-        </xacro:if>
         <jointName>
             steer_fl_joint, steer_fr_joint, wheel_fl_joint, wheel_fr_joint, wheel_rl_joint, wheel_rr_joint
         </jointName>
         <updateRate>100</updateRate>
-        <alwaysOn>true</alwaysOn>
     </plugin>
   </gazebo>

Commit message: Removed joint effort and velocity limits

File: audibot_description/urdf/audibot.urdf.xacro (robot description, xacro)
@@ -52,5 +52,5 @@
       <origin xyz="${x} ${y} ${z}" rpy="-1.57079632679 0 0" />
       <axis xyz="0 0 1" />
-      <limit effort="1000.0" velocity="22.0" />
+      <limit effort="-1.0" velocity="-1.0" />
     </joint>
   </xacro:macro>
@@ -86,5 +86,5 @@
       <origin xyz="${x} ${y} ${z}" rpy="0 0 0" />
       <axis xyz="0 0 1" />
-      <limit upper="0.6" lower="-0.6" effort="0.0" velocity="0.0" />
+      <limit upper="0.6" lower="-0.6" effort="-1.0" velocity="-1.0" />
     </joint>
     <joint name="wheel_${name}_joint" type="continuous" >
@@ -93,5 +93,5 @@
       <origin xyz="0 0 0" rpy="-1.57079632679 0 0" />
       <axis xyz="0 0 1" />
-      <limit effort="1000.0" velocity="22.0" />
+      <limit effort="-1.0" velocity="-1.0" />
     </joint>
   </xacro:macro>

Commit message: front axle

File: audibot_description/urdf/audibot.urdf.xacro (robot description, xacro)
@@ -127,4 +127,15 @@
     <child link="base_link"/>
   </joint>
+  <link name="front_axle">
+    <inertial>
+      <mass value="0.1"/>
+      <inertia ixx="0.0001" ixy="0.0001" ixz="0.0001" iyy="0.0001" iyz="0.0001" izz="0.0001" />
+    </inertial>
+  </link>
+  <joint name="front_axle_joint" type="fixed">
+    <origin xyz="${2*half_wheelbase} 0 0" rpy="0 0 0"/>
+    <parent link="base_footprint"/>
+    <child link="front_axle"/>
+  </joint>
   <xacro:rear_wheel name="rl" x="${-half_wheelbase}" y="${half_rear_track_width}" z="0" flip="1" />
   <xacro:rear_wheel name="rr" x="${-half_wheelbase}" y="${-half_rear_track_width}" z="0" flip="0" />
@@ -152,3 +163,7 @@
     <mu2>${wheel_friction}</mu2>
   </gazebo>
+  <!-- prevent fixed joint reduction -->
+  <gazebo reference="front_axle_joint" >
+    <preserveFixedJoint>true</preserveFixedJoint>
+  </gazebo>
 </robot>

Commit message: removed front_axle

File: audibot_description/urdf/audibot.urdf.xacro (robot description, xacro)
@@ -127,15 +127,4 @@
     <child link="base_link"/>
   </joint>
-  <link name="front_axle">
-    <inertial>
-      <mass value="0.1"/>
-      <inertia ixx="0.0001" ixy="0.0001" ixz="0.0001" iyy="0.0001" iyz="0.0001" izz="0.0001" />
-    </inertial>
-  </link>
-  <joint name="front_axle_joint" type="fixed">
-    <origin xyz="${2*half_wheelbase} 0 0" rpy="0 0 0"/>
-    <parent link="base_footprint"/>
-    <child link="front_axle"/>
-  </joint>
   <xacro:rear_wheel name="rl" x="${-half_wheelbase}" y="${half_rear_track_width}" z="0" flip="1" />
   <xacro:rear_wheel name="rr" x="${-half_wheelbase}" y="${-half_rear_track_width}" z="0" flip="0" />
@@ -163,7 +152,3 @@
     <mu2>${wheel_friction}</mu2>
   </gazebo>
-  <!-- prevent fixed joint reduction -->
-  <gazebo reference="front_axle_joint" >
-    <preserveFixedJoint>true</preserveFixedJoint>
-  </gazebo>
 </robot>

Commit message: Direct port to ROS 2

File: audibot_description/urdf/audibot.urdf.xacro (robot description, xacro)
@@ -13,17 +13,27 @@
   <xacro:arg name="pub_tf" default="true" />
   <xacro:arg name="robot_name" default="" />
+  <xacro:arg name="blue" default="false" />
   <gazebo>
     <!-- Simulated vehicle interface -->
     <plugin name="audibot_interface_plugin" filename="libaudibot_interface_plugin.so" >
-      <robotName>$(arg robot_name)</robotName>
-      <pubTf>$(arg pub_tf)</pubTf>
-      <tfFreq>100.0</tfFreq>
+      <robot_name>$(arg robot_name)</robot_name>
+      <pub_tf>$(arg pub_tf)</pub_tf>
+      <tf_freq>100.0</tf_freq>
+      <ros>
+        <namespace>$(arg robot_name)</namespace>
+      </ros>
     </plugin>
     <!-- Publish current joint angles -->
     <plugin name="joint_state_publisher" filename="libgazebo_ros_joint_state_publisher.so">
-        <jointName>
-            steer_fl_joint, steer_fr_joint, wheel_fl_joint, wheel_fr_joint, wheel_rl_joint, wheel_rr_joint
-        </jointName>
+        <joint_name>steer_fl_joint</joint_name>
+        <joint_name>steer_fr_joint</joint_name>
+        <joint_name>wheel_fl_joint</joint_name>
+        <joint_name>wheel_fr_joint</joint_name>
+        <joint_name>wheel_rl_joint</joint_name>
+        <joint_name>wheel_rr_joint</joint_name>
         <updateRate>100</updateRate>
+        <ros>
+          <namespace>$(arg robot_name)</namespace>
+        </ros>
     </plugin>
   </gazebo>
@@ -33,5 +43,5 @@
         <origin xyz="0 0 0" rpy="1.57079632679 ${flip * 3.1415926535} 0" />
         <geometry>
-          <mesh filename="package://audibot_description/meshes/wheel.dae" scale="1 1 1" />
+          <mesh filename="file://$(find audibot_description)/meshes/wheel.dae" scale="1 1 1" />
         </geometry>
       </visual>
@@ -60,5 +70,5 @@
         <origin xyz="0 0 0" rpy="1.57079632679 ${flip * pi} 0" />
         <geometry>
-          <mesh filename="package://audibot_description/meshes/wheel.dae" scale="1 1 1" />
+          <mesh filename="file://$(find audibot_description)/meshes/wheel.dae" scale="1 1 1" />
         </geometry>
       </visual>
@@ -103,8 +113,8 @@
       <geometry>
         <xacro:if value="$(arg blue)" >
-          <mesh filename="package://audibot_description/meshes/blue_body.dae" scale="1 1 1" />
+          <mesh filename="file://$(find audibot_description)/meshes/blue_body.dae" scale="1 1 1" />
         </xacro:if>
         <xacro:unless value="$(arg blue)" >
-          <mesh filename="package://audibot_description/meshes/orange_body.dae" scale="1 1 1" />
+          <mesh filename="file://$(find audibot_description)/meshes/orange_body.dae" scale="1 1 1" />
         </xacro:unless>
       </geometry>
@@ -113,5 +123,5 @@
       <origin xyz="0.035 0 0.025" rpy="0 0 0" />
       <geometry>
-        <mesh filename="package://audibot_description/meshes/body_collision.stl" scale="1 1 1" />
+        <mesh filename="file://$(find audibot_description)/meshes/body_collision.stl" scale="1 1 1" />
       </geometry>
     </collision>
